Commit message: feat(assets): migrate diagonal stations to TacCap assemblies
- Replace the xense-description diagonal-07/08 assemblies with TacCap
  variants (assembly/README/COMPONENTS .taccap, start_pose config).
- Add the TacCap slave gripper and Franka-to-TacCap tool adapter meshes.
- Use absolute controller joint angles in assembly and control chains;
  keep tool-finger mimic joints at a fixed viewer opening.
- Add identified TacCap URDFs and identification provenance.
- Record official CS66 source checks and conflicts.
- Assembly.viewer_joint_defaults() exposes viewer-only joint defaults.

File: libpyelite/assets/stations/diagonal-07/left_control.urdf (robot description, URDF)
Before this commit: robot cs66_left_absolute, 13 links, 12 joints
Joints:
- joint elbow_joint: origin xyz=-0.427 0 0 rpy=0 0 0 -> xyz=-0.427 0 0 rpy=0 -0 0
- joint shoulder_lift_joint: origin xyz=0 0 0 rpy=1.5707963265897931 0 0 -> xyz=0 0 0 rpy=1.5707963265897931 -0 0
- joint shoulder_pan_joint: origin xyz=0 0 0.1625 rpy=0 0 0 -> xyz=0 0 0.1625 rpy=0 -0 0
- joint wrist_1_joint: origin xyz=-0.3905 0 0.1475 rpy=0 0 0 -> xyz=-0.3905 0 0.1475 rpy=0 -0 0
- joint wrist_2_joint: origin xyz=0 -0.0965 0 rpy=1.5707963265897931 4.1530918500110381e-17 1.3479082663110799e-16 -> xyz=0 -0.0965 0 rpy=1.5707963265897931 -0 0
- joint wrist_3_joint: origin xyz=0 0.095 0 rpy=-1.5707963265897931 0 0 -> xyz=0 0.095 0 rpy=-1.5707963265897931 -0 0

File: libpyelite/assets/stations/diagonal-07/right_control.urdf (robot description, URDF)
Before this commit: robot cs66_right_absolute, 13 links, 12 joints
Joints:
- joint elbow_joint: origin xyz=-0.427 0 0 rpy=0 -0 1.5255279744540343e-16 -> xyz=-0.427 0 0 rpy=0 -0 0
- joint shoulder_lift_joint: origin xyz=0 0 0 rpy=1.5707963265897928 0 0 -> xyz=0 0 0 rpy=1.5707963265897931 -0 0
- joint shoulder_pan_joint: origin xyz=0 0 0.1625 rpy=0 0 0 -> xyz=0 0 0.1625 rpy=0 -0 0
- joint wrist_1_joint: origin xyz=-0.3905 0 0.1475 rpy=0 -0 1.4688354700645145e-17 -> xyz=-0.3905 0 0.1475 rpy=0 -0 0
- joint wrist_2_joint: origin xyz=0 -0.0965 0 rpy=1.5707963265897928 0 0 -> xyz=0 -0.0965 0 rpy=1.5707963265897931 -0 0
- joint wrist_3_joint: origin xyz=0 0.095 0 rpy=-1.5707963265897931 0 0 -> xyz=0 0.095 0 rpy=-1.5707963265897931 -0 0

File: libpyelite/assets/stations/source_assets/assemblies/diagonal-07-elite-cs66/urdf/diagonal-07-elite-cs66-taccap.urdf (robot description, URDF)
Before this commit: robot assembly_diagonal_08_elite_cs66, 31 links, 30 joints
Links:
- added link left_adapter_taccap_mount_link; collision mesh filename=../../../mounts/tool_adapters/flexiv_elite_franka_to_taccap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; visual mesh filename=../../../mounts/tool_adapters/flexiv_elite_franka_to_taccap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
- added link left_tool_taccap_base_link, mass 0.415; collision mesh filename=../../../grippers/xense/taccap/slave/body/meshes/base_link.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; visual mesh filename=../../../grippers/xense/taccap/slave/body/meshes/base_link.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
- added link left_tool_taccap_camera_link
- added link left_tool_taccap_camera_optical_link
- added link left_tool_taccap_eef_link
- added link left_tool_taccap_left_finger_link, mass 0.36678; collision mesh filename=../../../grippers/xense/taccap/slave/body/meshes/grip_left.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; visual mesh filename=../../../grippers/xense/taccap/slave/body/meshes/grip_left.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
- added link left_tool_taccap_right_finger_link, mass 0.36678; collision mesh filename=../../../grippers/xense/taccap/slave/body/meshes/grip_right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; visual mesh filename=../../../grippers/xense/taccap/slave/body/meshes/grip_right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
- added link right_adapter_taccap_mount_link; collision mesh filename=../../../mounts/tool_adapters/flexiv_elite_franka_to_taccap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; visual mesh filename=../../../mounts/tool_adapters/flexiv_elite_franka_to_taccap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
- added link right_tool_taccap_base_link, mass 0.415; collision mesh filename=../../../grippers/xense/taccap/slave/body/meshes/base_link.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; visual mesh filename=../../../grippers/xense/taccap/slave/body/meshes/base_link.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
- added link right_tool_taccap_camera_link
- added link right_tool_taccap_camera_optical_link
- added link right_tool_taccap_eef_link
- added link right_tool_taccap_left_finger_link, mass 0.36678; collision mesh filename=../../../grippers/xense/taccap/slave/body/meshes/grip_left.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; visual mesh filename=../../../grippers/xense/taccap/slave/body/meshes/grip_left.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
- added link right_tool_taccap_right_finger_link, mass 0.36678; collision mesh filename=../../../grippers/xense/taccap/slave/body/meshes/grip_right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; visual mesh filename=../../../grippers/xense/taccap/slave/body/meshes/grip_right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
Joints:
- added joint left_adapter_to_taccap_base: type fixed, parent left_adapter_taccap_mount_link, child left_tool_taccap_base_link, origin xyz=0 0 0.012 rpy=0 0 0
- added joint left_flange_to_taccap_adapter: type fixed, parent left_flange, child left_adapter_taccap_mount_link, origin xyz=0 0 0 rpy=0 0 0
- added joint left_tool_taccap_camera_joint: type fixed, parent left_tool_taccap_base_link, child left_tool_taccap_camera_link, origin xyz=-0.02275 0 0.06125 rpy=0 0 0
- added joint left_tool_taccap_camera_optical_joint: type fixed, parent left_tool_taccap_camera_link, child left_tool_taccap_camera_optical_link, origin xyz=0 0 0 rpy=0 0 -1.5707963267948966
- added joint left_tool_taccap_eef_joint: type fixed, parent left_tool_taccap_base_link, child left_tool_taccap_eef_link, origin xyz=0.036575 0 0.2009217 rpy=0 0 0
- added joint left_tool_taccap_left_finger_joint: type revolute, parent left_tool_taccap_base_link, child left_tool_taccap_left_finger_link, origin xyz=0.0120336718 0.0199500106 0.0484999712 rpy=0 0 0, axis 1 0 0, limit lower=-0.5047492196767601 upper=0 effort=4 velocity=1, mimic joint=left_tool_taccap_right_finger_joint multiplier=-1 offset=0
- added joint left_tool_taccap_right_finger_joint: type revolute, parent left_tool_taccap_base_link, child left_tool_taccap_right_finger_link, origin xyz=0.0120336718 -0.0199499894 0.0484999712 rpy=0 0 0, axis 1 0 0, limit lower=0 upper=0.5047492196767601 effort=4 velocity=1
- added joint right_adapter_to_taccap_base: type fixed, parent right_adapter_taccap_mount_link, child right_tool_taccap_base_link, origin xyz=0 0 0.012 rpy=0 0 0
- added joint right_flange_to_taccap_adapter: type fixed, parent right_flange, child right_adapter_taccap_mount_link, origin xyz=0 0 0 rpy=0 0 -1.5707963267948966
- added joint right_tool_taccap_camera_joint: type fixed, parent right_tool_taccap_base_link, child right_tool_taccap_camera_link, origin xyz=-0.02275 0 0.06125 rpy=0 0 0
- added joint right_tool_taccap_camera_optical_joint: type fixed, parent right_tool_taccap_camera_link, child right_tool_taccap_camera_optical_link, origin xyz=0 0 0 rpy=0 0 -1.5707963267948966
- added joint right_tool_taccap_eef_joint: type fixed, parent right_tool_taccap_base_link, child right_tool_taccap_eef_link, origin xyz=0.036575 0 0.2009217 rpy=0 0 0
- added joint right_tool_taccap_left_finger_joint: type revolute, parent right_tool_taccap_base_link, child right_tool_taccap_left_finger_link, origin xyz=0.0120336718 0.0199500106 0.0484999712 rpy=0 0 0, axis 1 0 0, limit lower=-0.5047492196767601 upper=0 effort=4 velocity=1, mimic joint=right_tool_taccap_right_finger_joint multiplier=-1 offset=0
- added joint right_tool_taccap_right_finger_joint: type revolute, parent right_tool_taccap_base_link, child right_tool_taccap_right_finger_link, origin xyz=0.0120336718 -0.0199499894 0.0484999712 rpy=0 0 0, axis 1 0 0, limit lower=0 upper=0.5047492196767601 effort=4 velocity=1
- joint left_elbow_joint: limit lower=-4.7123926535897933 upper=1.5707926535897931 effort=150.0 velocity=3.141592653589793 -> lower=-3.141592653589793 upper=3.141592653589793 effort=150.0 velocity=3.141592653589793; origin xyz=-0.427 0 0 rpy=0 -0 1.5708 -> xyz=-0.427 0 0 rpy=0 0 0
- joint left_shoulder_lift_joint: limit lower=-5.7595853071795862 upper=6.8067853071795863 effort=150.0 velocity=3.141592653589793 -> lower=-6.283185307179586 upper=6.283185307179586 effort=150.0 velocity=3.141592653589793; origin xyz=0 0 0 rpy=1.5707963265580633 0.52359999999999995 -1.184169252091432e-10 -> xyz=0 0 0 rpy=1.570796326589793 0 0
- joint left_shoulder_pan_joint: limit lower=-4.8868853071795861 upper=7.6794853071795863 effort=150.0 velocity=3.141592653589793 -> lower=-6.283185307179586 upper=6.283185307179586 effort=150.0 velocity=3.141592653589793; origin xyz=0 0 0.1625 rpy=0 -0 -1.3963000000000001 -> xyz=0 0 0.1625 rpy=0 0 0
- joint left_wrist_1_joint: limit lower=-5.7595853071795862 upper=6.8067853071795863 effort=28.0 velocity=3.141592653589793 -> lower=-6.283185307179586 upper=6.283185307179586 effort=28.0 velocity=3.141592653589793; origin xyz=-0.3905 0 0.1475 rpy=0 -0 -0.52359999999999995 -> xyz=-0.3905 0 0.1475 rpy=0 0 0
- joint left_wrist_2_joint: limit lower=-7.8539853071795864 upper=4.712385307179586 effort=28.0 velocity=3.141592653589793 -> lower=-6.283185307179586 upper=6.283185307179586 effort=28.0 velocity=3.141592653589793; origin xyz=0 -0.0965 0 rpy=-1.5707404890333243 -1.5707926535897876 3.1415368158282213 -> xyz=0 -0.0965 0 rpy=1.570796326589793 0 0
- joint left_wrist_3_joint: limit lower=-5.4977853071795861 upper=7.0685853071795863 effort=28.0 velocity=3.141592653589793 -> lower=-6.283185307179586 upper=6.283185307179586 effort=28.0 velocity=3.141592653589793; origin xyz=0 0.095 0 rpy=-1.5707963265048359 -0.78539999999999999 -2.0510430436880494e-10 -> xyz=0 0.095 0 rpy=-1.570796326589793 0 0
- joint right_elbow_joint: limit lower=-1.5707926535897931 upper=4.7123926535897933 effort=150.0 velocity=3.141592653589793 -> lower=-3.141592653589793 upper=3.141592653589793 effort=150.0 velocity=3.141592653589793; origin xyz=-0.427 0 0 rpy=0 -0 -1.5708 -> xyz=-0.427 0 0 rpy=0 0 0
- joint right_shoulder_lift_joint: limit lower=-3.6651853071795863 upper=8.9011853071795866 effort=150.0 velocity=3.141592653589793 -> lower=-6.283185307179586 upper=6.283185307179586 effort=150.0 velocity=3.141592653589793; origin xyz=0 0 0 rpy=-1.5707963265580642 0.52359265358979334 -3.1415926534713785 -> xyz=0 0 0 rpy=1.570796326589793 0 0
- joint right_shoulder_pan_joint: limit lower=-4.5378853071795859 upper=8.0284853071795865 effort=150.0 velocity=3.141592653589793 -> lower=-6.283185307179586 upper=6.283185307179586 effort=150.0 velocity=3.141592653589793; origin xyz=0 0 0.1625 rpy=0 -0 -1.7453000000000001 -> xyz=0 0 0.1625 rpy=0 0 0
- joint right_wrist_1_joint: limit lower=-3.6651853071795863 upper=8.9011853071795866 effort=28.0 velocity=3.141592653589793 -> lower=-6.283185307179586 upper=6.283185307179586 effort=28.0 velocity=3.141592653589793; origin xyz=-0.3905 0 0.1475 rpy=0 -0 -2.6179999999999999 -> xyz=-0.3905 0 0.1475 rpy=0 0 0
- joint right_wrist_2_joint: limit lower=-4.712385307179586 upper=7.8539853071795864 effort=28.0 velocity=3.141592653589793 -> lower=-6.283185307179586 upper=6.283185307179586 effort=28.0 velocity=3.141592653589793; origin xyz=0 -0.0965 0 rpy=-1.5707404890333243 1.5707926535897876 -3.1415368158282213 -> xyz=0 -0.0965 0 rpy=1.570796326589793 0 0
- joint right_wrist_3_joint: limit lower=-5.4977853071795861 upper=7.0685853071795863 effort=28.0 velocity=3.141592653589793 -> lower=-6.283185307179586 upper=6.283185307179586 effort=28.0 velocity=3.141592653589793; origin xyz=0 0.095 0 rpy=-1.5707963265048359 -0.78539999999999999 -2.0510430436880494e-10 -> xyz=0 0.095 0 rpy=-1.570796326589793 0 0
- joint world_to_table: origin xyz=0.700624760246217 -0.0677769600617899 0.000895483271931539 rpy=0 0 0 -> xyz=0.700624760246217 0.067776960061789945 0.000895483271931539 rpy=0 0 0

File: libpyelite/assets/stations/source_assets/assemblies/diagonal-08-elite-cs66/urdf/diagonal-08-elite-cs66-taccap.urdf (robot description, URDF)
Before this commit: robot assembly_diagonal_07_elite_cs66, 31 links, 30 joints
Links:
- added link left_adapter_taccap_mount_link; collision mesh filename=../../../mounts/tool_adapters/flexiv_elite_franka_to_taccap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; visual mesh filename=../../../mounts/tool_adapters/flexiv_elite_franka_to_taccap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
- added link left_tool_taccap_base_link, mass 0.415; collision mesh filename=../../../grippers/xense/taccap/slave/body/meshes/base_link.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; visual mesh filename=../../../grippers/xense/taccap/slave/body/meshes/base_link.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
- added link left_tool_taccap_camera_link
- added link left_tool_taccap_camera_optical_link
- added link left_tool_taccap_eef_link
- added link left_tool_taccap_left_finger_link, mass 0.36678; collision mesh filename=../../../grippers/xense/taccap/slave/body/meshes/grip_left.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; visual mesh filename=../../../grippers/xense/taccap/slave/body/meshes/grip_left.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
- added link left_tool_taccap_right_finger_link, mass 0.36678; collision mesh filename=../../../grippers/xense/taccap/slave/body/meshes/grip_right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; visual mesh filename=../../../grippers/xense/taccap/slave/body/meshes/grip_right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
- added link right_adapter_taccap_mount_link; collision mesh filename=../../../mounts/tool_adapters/flexiv_elite_franka_to_taccap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; visual mesh filename=../../../mounts/tool_adapters/flexiv_elite_franka_to_taccap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
- added link right_tool_taccap_base_link, mass 0.415; collision mesh filename=../../../grippers/xense/taccap/slave/body/meshes/base_link.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; visual mesh filename=../../../grippers/xense/taccap/slave/body/meshes/base_link.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
- added link right_tool_taccap_camera_link
- added link right_tool_taccap_camera_optical_link
- added link right_tool_taccap_eef_link
- added link right_tool_taccap_left_finger_link, mass 0.36678; collision mesh filename=../../../grippers/xense/taccap/slave/body/meshes/grip_left.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; visual mesh filename=../../../grippers/xense/taccap/slave/body/meshes/grip_left.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
- added link right_tool_taccap_right_finger_link, mass 0.36678; collision mesh filename=../../../grippers/xense/taccap/slave/body/meshes/grip_right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; visual mesh filename=../../../grippers/xense/taccap/slave/body/meshes/grip_right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
Joints:
- added joint left_adapter_to_taccap_base: type fixed, parent left_adapter_taccap_mount_link, child left_tool_taccap_base_link, origin xyz=0 0 0.012 rpy=0 0 0
- added joint left_flange_to_taccap_adapter: type fixed, parent left_flange, child left_adapter_taccap_mount_link, origin xyz=0 0 0 rpy=0 0 0
- added joint left_tool_taccap_camera_joint: type fixed, parent left_tool_taccap_base_link, child left_tool_taccap_camera_link, origin xyz=-0.02275 0 0.06125 rpy=0 0 0
- added joint left_tool_taccap_camera_optical_joint: type fixed, parent left_tool_taccap_camera_link, child left_tool_taccap_camera_optical_link, origin xyz=0 0 0 rpy=0 0 -1.5707963267948966
- added joint left_tool_taccap_eef_joint: type fixed, parent left_tool_taccap_base_link, child left_tool_taccap_eef_link, origin xyz=0.036575 0 0.2009217 rpy=0 0 0
- added joint left_tool_taccap_left_finger_joint: type revolute, parent left_tool_taccap_base_link, child left_tool_taccap_left_finger_link, origin xyz=0.0120336718 0.0199500106 0.0484999712 rpy=0 0 0, axis 1 0 0, limit lower=-0.5047492196767601 upper=0 effort=4 velocity=1, mimic joint=left_tool_taccap_right_finger_joint multiplier=-1 offset=0
- added joint left_tool_taccap_right_finger_joint: type revolute, parent left_tool_taccap_base_link, child left_tool_taccap_right_finger_link, origin xyz=0.0120336718 -0.0199499894 0.0484999712 rpy=0 0 0, axis 1 0 0, limit lower=0 upper=0.5047492196767601 effort=4 velocity=1
- added joint right_adapter_to_taccap_base: type fixed, parent right_adapter_taccap_mount_link, child right_tool_taccap_base_link, origin xyz=0 0 0.012 rpy=0 0 0
- added joint right_flange_to_taccap_adapter: type fixed, parent right_flange, child right_adapter_taccap_mount_link, origin xyz=0 0 0 rpy=0 0 -1.5707963267948966
- added joint right_tool_taccap_camera_joint: type fixed, parent right_tool_taccap_base_link, child right_tool_taccap_camera_link, origin xyz=-0.02275 0 0.06125 rpy=0 0 0
- added joint right_tool_taccap_camera_optical_joint: type fixed, parent right_tool_taccap_camera_link, child right_tool_taccap_camera_optical_link, origin xyz=0 0 0 rpy=0 0 -1.5707963267948966
- added joint right_tool_taccap_eef_joint: type fixed, parent right_tool_taccap_base_link, child right_tool_taccap_eef_link, origin xyz=0.036575 0 0.2009217 rpy=0 0 0
- added joint right_tool_taccap_left_finger_joint: type revolute, parent right_tool_taccap_base_link, child right_tool_taccap_left_finger_link, origin xyz=0.0120336718 0.0199500106 0.0484999712 rpy=0 0 0, axis 1 0 0, limit lower=-0.5047492196767601 upper=0 effort=4 velocity=1, mimic joint=right_tool_taccap_right_finger_joint multiplier=-1 offset=0
- added joint right_tool_taccap_right_finger_joint: type revolute, parent right_tool_taccap_base_link, child right_tool_taccap_right_finger_link, origin xyz=0.0120336718 -0.0199499894 0.0484999712 rpy=0 0 0, axis 1 0 0, limit lower=0 upper=0.5047492196767601 effort=4 velocity=1
- joint left_elbow_joint: limit lower=-4.7123926535897933 upper=1.5707926535897931 effort=150.0 velocity=3.141592653589793 -> lower=-3.141592653589793 upper=3.141592653589793 effort=150.0 velocity=3.141592653589793; origin xyz=-0.427 0 0 rpy=0 -0 1.5708 -> xyz=-0.427 0 0 rpy=0 0 0
- joint left_shoulder_lift_joint: limit lower=-5.7595853071795862 upper=6.8067853071795863 effort=150.0 velocity=3.141592653589793 -> lower=-6.283185307179586 upper=6.283185307179586 effort=150.0 velocity=3.141592653589793; origin xyz=0 0 0 rpy=1.5707963265580633 0.52359999999999995 -1.184169252091432e-10 -> xyz=0 0 0 rpy=1.570796326589793 0 0
- joint left_shoulder_pan_joint: limit lower=-4.8868853071795861 upper=7.6794853071795863 effort=150.0 velocity=3.141592653589793 -> lower=-6.283185307179586 upper=6.283185307179586 effort=150.0 velocity=3.141592653589793; origin xyz=0 0 0.1625 rpy=0 -0 -1.3963000000000001 -> xyz=0 0 0.1625 rpy=0 0 0
- joint left_wrist_1_joint: limit lower=-5.7595853071795862 upper=6.8067853071795863 effort=28.0 velocity=3.141592653589793 -> lower=-6.283185307179586 upper=6.283185307179586 effort=28.0 velocity=3.141592653589793; origin xyz=-0.3905 0 0.1475 rpy=0 -0 -0.52359999999999995 -> xyz=-0.3905 0 0.1475 rpy=0 0 0
- joint left_wrist_2_joint: limit lower=-7.8539853071795864 upper=4.712385307179586 effort=28.0 velocity=3.141592653589793 -> lower=-6.283185307179586 upper=6.283185307179586 effort=28.0 velocity=3.141592653589793; origin xyz=0 -0.0965 0 rpy=-1.5707404890333243 -1.5707926535897876 3.1415368158282213 -> xyz=0 -0.0965 0 rpy=1.570796326589793 0 0
- joint left_wrist_3_joint: limit lower=-5.4977853071795861 upper=7.0685853071795863 effort=28.0 velocity=3.141592653589793 -> lower=-6.283185307179586 upper=6.283185307179586 effort=28.0 velocity=3.141592653589793; origin xyz=0 0.095 0 rpy=-1.5707963265048359 -0.78539999999999999 -2.0510430436880494e-10 -> xyz=0 0.095 0 rpy=-1.570796326589793 0 0
- joint right_elbow_joint: limit lower=-1.5707926535897931 upper=4.7123926535897933 effort=150.0 velocity=3.141592653589793 -> lower=-3.141592653589793 upper=3.141592653589793 effort=150.0 velocity=3.141592653589793; origin xyz=-0.427 0 0 rpy=0 -0 -1.5708 -> xyz=-0.427 0 0 rpy=0 0 0
- joint right_shoulder_lift_joint: limit lower=-3.6651853071795863 upper=8.9011853071795866 effort=150.0 velocity=3.141592653589793 -> lower=-6.283185307179586 upper=6.283185307179586 effort=150.0 velocity=3.141592653589793; origin xyz=0 0 0 rpy=-1.5707963265580642 0.52359265358979334 -3.1415926534713785 -> xyz=0 0 0 rpy=1.570796326589793 0 0
- joint right_shoulder_pan_joint: limit lower=-4.5378853071795859 upper=8.0284853071795865 effort=150.0 velocity=3.141592653589793 -> lower=-6.283185307179586 upper=6.283185307179586 effort=150.0 velocity=3.141592653589793; origin xyz=0 0 0.1625 rpy=0 -0 -1.7453000000000001 -> xyz=0 0 0.1625 rpy=0 0 0
- joint right_wrist_1_joint: limit lower=-3.6651853071795863 upper=8.9011853071795866 effort=28.0 velocity=3.141592653589793 -> lower=-6.283185307179586 upper=6.283185307179586 effort=28.0 velocity=3.141592653589793; origin xyz=-0.3905 0 0.1475 rpy=0 -0 -2.6179999999999999 -> xyz=-0.3905 0 0.1475 rpy=0 0 0
- joint right_wrist_2_joint: limit lower=-4.712385307179586 upper=7.8539853071795864 effort=28.0 velocity=3.141592653589793 -> lower=-6.283185307179586 upper=6.283185307179586 effort=28.0 velocity=3.141592653589793; origin xyz=0 -0.0965 0 rpy=-1.5707404890333243 1.5707926535897876 -3.1415368158282213 -> xyz=0 -0.0965 0 rpy=1.570796326589793 0 0
- joint right_wrist_3_joint: limit lower=-5.4977853071795861 upper=7.0685853071795863 effort=28.0 velocity=3.141592653589793 -> lower=-6.283185307179586 upper=6.283185307179586 effort=28.0 velocity=3.141592653589793; origin xyz=0 0.095 0 rpy=-1.5707963265048359 -0.78539999999999999 -2.0510430436880494e-10 -> xyz=0 0.095 0 rpy=-1.570796326589793 0 0
- joint world_to_table: origin xyz=0.700624760246217 -0.0677769600617899 0.000895483271931539 rpy=0 0 0 -> xyz=0.700624760246217 0.067776960061789945 0.000895483271931539 rpy=0 0 0
